Commit message: Updated robot model.

File: Project2/catkin_ws/src/my_robot/urdf/my_robot.xacro (robot description, xacro)
@@ -9,5 +9,5 @@
   </joint>
   <link name='chassis'>
-    <pose>0 0 0.1 0 0 0</pose>
+    <pose>0 0 0.03 0 0 0</pose>
     <inertial>
       <mass value="15.0"/>
@@ -28,9 +28,9 @@
       <origin xyz="0 0 0" rpy=" 0 0 0"/>
       <geometry>
-        <box size=".4 .2 .1"/>
+        <cylinder radius="0.25" length="0.1"/>
       </geometry>
     </visual>
     <collision name='back_caster_collision'>
-      <origin xyz="-0.15 0 -0.05" rpy=" 0 0 0"/>
+      <origin xyz="-0.15 0 -0.03" rpy=" 0 0 0"/>
       <geometry>
         <sphere radius="0.0499"/>
@@ -38,5 +38,5 @@
     </collision>
     <visual name='back_caster_visual'>
-      <origin xyz="-0.15 0 -0.05" rpy=" 0 0 0"/>
+      <origin xyz="-0.15 0 -0.03" rpy=" 0 0 0"/>
       <geometry>
         <sphere radius="0.05"/>
@@ -44,5 +44,5 @@
     </visual>
     <collision name='front_caster_collision'>
-      <origin xyz="0.15 0 -0.05" rpy=" 0 0 0"/>
+      <origin xyz="0.15 0 -0.03" rpy=" 0 0 0"/>
       <geometry>
         <sphere radius="0.0499"/>
@@ -50,5 +50,5 @@
     </collision>
     <visual name='front_caster_visual'>
-      <origin xyz="0.15 0 -0.05" rpy=" 0 0 0"/>
+      <origin xyz="0.15 0 -0.03" rpy=" 0 0 0"/>
       <geometry>
         <sphere radius="0.05"/>
@@ -56,4 +56,7 @@
     </visual>
   </link>
+  <gazebo reference="chassis">
+    <material>Gazebo/Orange</material>
+  </gazebo>
   <link name="left_wheel">
     <pose>0 0 0 0 0 0</pose>
@@ -70,5 +73,5 @@
       <origin xyz="0 0 0" rpy=" 0 1.5707 1.5707"/>
       <geometry>
-        <cylinder radius=".1" length="0.05"/>
+        <cylinder radius=".05" length="0.05"/>
       </geometry>
     </collision>
@@ -76,13 +79,13 @@
       <origin xyz="0 0 0" rpy=" 0 1.5707 1.5707"/>
       <geometry>
-        <cylinder radius=".1" length="0.05"/>
+        <cylinder radius=".05" length="0.05"/>
       </geometry>
     </visual>
   </link>
   <gazebo reference="left_wheel">
-    <material>Gazebo/Green</material>
+    <material>Gazebo/Blue</material>
   </gazebo>
   <joint type="continuous" name="left_wheel_hinge">
-    <origin xyz="0 0.15 0" rpy="0 0 0"/>
+    <origin xyz="0 0.18 -0.03" rpy="0 0 0"/>
     <child link="left_wheel"/>
     <parent link="chassis"/>
@@ -105,5 +108,5 @@
       <origin xyz="0 0 0" rpy=" 0 1.5707 1.5707"/>
       <geometry>
-        <cylinder radius=".1" length="0.05"/>
+        <cylinder radius=".05" length="0.05"/>
       </geometry>
     </collision>
@@ -111,13 +114,13 @@
       <origin xyz="0 0 0" rpy=" 0 1.5707 1.5707"/>
       <geometry>
-        <cylinder radius=".1" length="0.05"/>
+        <cylinder radius=".05" length="0.05"/>
       </geometry>
     </visual>
   </link>
   <gazebo reference="right_wheel">
-    <material>Gazebo/Green</material>
+    <material>Gazebo/Blue</material>
   </gazebo>
   <joint type="continuous" name="right_wheel_hinge">
-    <origin xyz="0 -0.15 0" rpy="0 0 0"/>
+    <origin xyz="0 -0.18 -0.03" rpy="0 0 0"/>
     <child link="right_wheel"/>
     <parent link="chassis"/>
@@ -154,5 +157,5 @@
   </gazebo>
   <joint type="fixed" name="camera_joint">
-    <origin xyz="0.2 0 0" rpy="0 0 0"/>
+    <origin xyz="0.2 -0.05 0" rpy="0 0 0"/>
     <child link="camera"/>
     <parent link="chassis"/>
@@ -184,5 +187,5 @@
   </link>
   <joint type="fixed" name="hokuyo_joint">
-    <origin xyz="0.15 0 0.1" rpy="0 0 0"/>
+    <origin xyz="0.2 0.05 0" rpy="0 0 0"/>
     <child link="hokuyo"/>
     <parent link="chassis"/>
